Commit message: feat: add tracked differential simulation control

File: src/carbot_description/urdf/carbot.urdf.xacro (robot description, xacro)
@@ -105,5 +105,9 @@
       <child link="${side}_${group}_wheel_link"/>
       <origin xyz="${wheel['x_m']} ${y} ${wheel['z_m']}" rpy="0 0 0"/>
-      <axis xyz="0 1 0"/>
+      <!-- -Y makes positive joint velocity move either track toward +X. -->
+      <axis xyz="0 -1 0"/>
+      <limit
+        effort="${p['dynamics']['per_side_effort_limit_nm'] / 6.0}"
+        velocity="${p['control']['max_wheel_velocity_rad_s']}"/>
       <dynamics damping="${p['dynamics']['joint_damping_nm_s_rad']}" friction="0"/>
     </joint>

Commit message: fix: remove legacy carter and expose tracks

File: src/carbot_description/urdf/carbot.urdf.xacro (robot description, xacro)
@@ -4,4 +4,5 @@
   <xacro:property name="p" value="${xacro.load_yaml('$(arg parameters_file)')}"/>
   <xacro:property name="body" value="${p['geometry']['body_collision']}"/>
+  <xacro:property name="body_visual" value="${p['geometry']['body_visual']}"/>
   <xacro:property name="wheels" value="${p['geometry']['wheel_groups']}"/>
   <xacro:property name="track_y" value="${p['geometry']['physical_track_separation_m'] / 2.0}"/>
@@ -39,7 +40,7 @@
     </inertial>
     <visual name="body_visual">
-      <origin xyz="${body['position_from_base_link_m'][0]} ${body['position_from_base_link_m'][1]} ${body['position_from_base_link_m'][2]}" rpy="0 0 0"/>
+      <origin xyz="${body_visual['position_from_base_link_m'][0]} ${body_visual['position_from_base_link_m'][1]} ${body_visual['position_from_base_link_m'][2]}" rpy="0 0 0"/>
       <geometry>
-        <box size="${body['size_m'][0]} ${body['size_m'][1]} ${body['size_m'][2]}"/>
+        <box size="${body_visual['size_m'][0]} ${body_visual['size_m'][1]} ${body_visual['size_m'][2]}"/>
       </geometry>
       <material name="carbot_blue"/>

Commit message: fix: add visible mid360 mounting support

File: src/carbot_description/urdf/carbot.urdf.xacro (robot description, xacro)
@@ -14,4 +14,7 @@
   <xacro:property name="track_top_z" value="${wheels['front_idler']['z_m'] + wheels['front_idler']['radius_m']}"/>
   <xacro:property name="wheel_mass" value="${p['dynamics']['per_wheel_mass_kg']}"/>
+  <xacro:property name="body_visual_top_z" value="${body_visual['position_from_base_link_m'][2] + body_visual['size_m'][2] / 2.0}"/>
+  <xacro:property name="lidar_origin_z" value="${p['sensors']['mid360']['translation_from_base_link_m'][2]}"/>
+  <xacro:property name="lidar_mount_height" value="${lidar_origin_z - body_visual_top_z}"/>
   <material name="carbot_blue">
     <color rgba="0.08 0.24 0.55 1.0"/>
@@ -129,4 +132,14 @@
   <xacro:wheel side="right" group="rear_drive" y="${-track_y}"/>
   <link name="lidar_link">
+    <!-- Design proxy only: fills the visible mounting space without changing the measured lidar origin. -->
+    <visual name="mid360_mount_proxy_visual">
+      <origin xyz="0 0 ${-lidar_mount_height / 2.0}" rpy="0 0 0"/>
+      <geometry>
+        <cylinder
+          radius="${p['sensors']['mid360']['mount_proxy']['radius_m']}"
+          length="${lidar_mount_height}"/>
+      </geometry>
+      <material name="sensor_gray"/>
+    </visual>
     <visual name="mid360_proxy_visual">
       <origin xyz="0 0 0.02" rpy="0 0 0"/>

Commit message: fix: model measured mid360 housing height

File: src/carbot_description/urdf/carbot.urdf.xacro (robot description, xacro)
@@ -14,7 +14,6 @@
   <xacro:property name="track_top_z" value="${wheels['front_idler']['z_m'] + wheels['front_idler']['radius_m']}"/>
   <xacro:property name="wheel_mass" value="${p['dynamics']['per_wheel_mass_kg']}"/>
-  <xacro:property name="body_visual_top_z" value="${body_visual['position_from_base_link_m'][2] + body_visual['size_m'][2] / 2.0}"/>
-  <xacro:property name="lidar_origin_z" value="${p['sensors']['mid360']['translation_from_base_link_m'][2]}"/>
-  <xacro:property name="lidar_mount_height" value="${lidar_origin_z - body_visual_top_z}"/>
+  <xacro:property name="lidar_housing_height" value="${p['sensors']['mid360']['housing_height_m']}"/>
+  <xacro:property name="lidar_mount_z" value="${p['sensors']['mid360']['housing_top_height_from_ground_m'] - lidar_housing_height - p['geometry']['base_link_height_m']}"/>
   <material name="carbot_blue">
     <color rgba="0.08 0.24 0.55 1.0"/>
@@ -132,20 +131,10 @@
   <xacro:wheel side="right" group="rear_drive" y="${-track_y}"/>
   <link name="lidar_link">
-    <!-- Design proxy only: fills the visible mounting space without changing the measured lidar origin. -->
-    <visual name="mid360_mount_proxy_visual">
-      <origin xyz="0 0 ${-lidar_mount_height / 2.0}" rpy="0 0 0"/>
-      <geometry>
-        <cylinder
-          radius="${p['sensors']['mid360']['mount_proxy']['radius_m']}"
-          length="${lidar_mount_height}"/>
-      </geometry>
-      <material name="sensor_gray"/>
-    </visual>
     <visual name="mid360_proxy_visual">
-      <origin xyz="0 0 0.02" rpy="0 0 0"/>
+      <origin xyz="0 0 ${lidar_housing_height / 2.0}" rpy="0 0 0"/>
       <geometry>
         <cylinder
           radius="${p['sensors']['mid360']['visual_proxy']['radius_m']}"
-          length="${p['sensors']['mid360']['visual_proxy']['height_m']}"/>
+          length="${lidar_housing_height}"/>
       </geometry>
       <material name="sensor_gray"/>
@@ -156,5 +145,5 @@
     <child link="lidar_link"/>
     <origin
-      xyz="${p['sensors']['mid360']['translation_from_base_link_m'][0]} ${p['sensors']['mid360']['translation_from_base_link_m'][1]} ${p['sensors']['mid360']['translation_from_base_link_m'][2]}"
+      xyz="${p['sensors']['mid360']['mount_translation_xy_from_base_link_m'][0]} ${p['sensors']['mid360']['mount_translation_xy_from_base_link_m'][1]} ${lidar_mount_z}"
       rpy="${p['sensors']['mid360']['rotation_rpy_rad'][0]} ${p['sensors']['mid360']['rotation_rpy_rad'][1]} ${p['sensors']['mid360']['rotation_rpy_rad'][2]}"/>
   </joint>

Commit message: feat: finalize Carbot real robot adaptation

File: src/carbot_description/urdf/carbot.urdf.xacro (robot description, xacro)
@@ -16,4 +16,5 @@
   <xacro:property name="lidar_housing_height" value="${p['sensors']['mid360']['housing_height_m']}"/>
   <xacro:property name="lidar_mount_z" value="${p['sensors']['mid360']['housing_top_height_from_ground_m'] - lidar_housing_height - p['geometry']['base_link_height_m']}"/>
+  <xacro:property name="livox_origin_z" value="${p['sensors']['mid360']['coordinate_origin_height_from_housing_bottom_m']}"/>
   <material name="carbot_blue">
     <color rgba="0.08 0.24 0.55 1.0"/>
@@ -151,10 +152,10 @@
   <joint name="lidar_link_to_livox_frame" type="fixed">
     <parent link="lidar_link"/><child link="livox_frame"/>
-    <origin xyz="0 0 0" rpy="0 0 0"/>
+    <origin xyz="0 0 ${livox_origin_z}" rpy="0 0 0"/>
   </joint>
   <link name="front_3d_lidar"/>
   <joint name="lidar_link_to_front_3d_lidar" type="fixed">
     <parent link="lidar_link"/><child link="front_3d_lidar"/>
-    <origin xyz="0 0 0" rpy="0 0 0"/>
+    <origin xyz="0 0 ${livox_origin_z}" rpy="0 0 0"/>
   </joint>
   <link name="imu_link"/>

Commit message: feat(isaac): add Carbot body, D455 mount and ToF array

File: src/carbot_description/urdf/carbot.urdf.xacro (robot description, xacro)
@@ -5,4 +5,5 @@
   <xacro:property name="body" value="${p['geometry']['body_collision']}"/>
   <xacro:property name="body_visual" value="${p['geometry']['body_visual']}"/>
+  <xacro:property name="body_visual_base_plate" value="${p['geometry']['body_visual_base_plate']}"/>
   <xacro:property name="wheels" value="${p['geometry']['wheel_groups']}"/>
   <xacro:property name="track_y" value="${p['geometry']['physical_track_separation_m'] / 2.0}"/>
@@ -19,4 +20,7 @@
   <material name="carbot_blue">
     <color rgba="0.08 0.24 0.55 1.0"/>
+  </material>
+  <material name="base_plate_green">
+    <color rgba="0.05 0.65 0.12 1.0"/>
   </material>
   <material name="track_black">
@@ -49,4 +53,11 @@
       <material name="carbot_blue"/>
     </visual>
+    <visual name="body_visual_base_plate">
+      <origin xyz="${body_visual_base_plate['position_from_base_link_m'][0]} ${body_visual_base_plate['position_from_base_link_m'][1]} ${body_visual_base_plate['position_from_base_link_m'][2]}" rpy="0 0 0"/>
+      <geometry>
+        <box size="${body_visual_base_plate['size_m'][0]} ${body_visual_base_plate['size_m'][1]} ${body_visual_base_plate['size_m'][2]}"/>
+      </geometry>
+      <material name="base_plate_green"/>
+    </visual>
     <collision name="body_collision">
       <origin xyz="${body['position_from_base_link_m'][0]} ${body['position_from_base_link_m'][1]} ${body['position_from_base_link_m'][2]}" rpy="0 0 0"/>
@@ -64,10 +75,10 @@
   <xacro:macro name="track_visual" params="side y">
     <link name="${side}_track_visual_link">
-      <visual name="lower_belt">
+      <visual name="${side}_lower_belt">
         <origin xyz="0 0 ${track_bottom_z}" rpy="0 0 0"/>
         <geometry><box size="${track_length} ${track_width} ${track_thickness}"/></geometry>
         <material name="track_black"/>
       </visual>
-      <visual name="upper_belt">
+      <visual name="${side}_upper_belt">
         <origin xyz="0 0 ${track_top_z}" rpy="0 0 0"/>
         <geometry><box size="${track_visual_length} ${track_width} ${track_thickness}"/></geometry>

Commit message: model carbot sensor mounts and measured body layout

File: src/carbot_description/urdf/carbot.urdf.xacro (robot description, xacro)
@@ -32,4 +32,13 @@
   <material name="sensor_gray">
     <color rgba="0.16 0.17 0.18 1.0"/>
+  </material>
+  <material name="mid360_mount_gray">
+    <color rgba="0.22 0.23 0.24 1.0"/>
+  </material>
+  <material name="mid360_body_gray">
+    <color rgba="0.10 0.11 0.12 1.0"/>
+  </material>
+  <material name="mid360_window_black">
+    <color rgba="0.015 0.02 0.025 1.0"/>
   </material>
   <link name="base_footprint"/>
@@ -143,12 +152,28 @@
   <xacro:wheel side="right" group="rear_drive" y="${-track_y}"/>
   <link name="lidar_link">
-    <visual name="mid360_proxy_visual">
-      <origin xyz="0 0 ${lidar_housing_height / 2.0}" rpy="0 0 0"/>
+    <!-- Visual-only MID-360 envelope. Sensor origins and physical parameters
+         remain defined by the fixed joints and canonical calibration above. -->
+    <visual name="mid360_mount_visual">
+      <origin xyz="0 0 ${p['sensors']['mid360']['visual_proxy']['mount_size_m'][2] / 2.0}" rpy="0 0 0"/>
+      <geometry>
+        <box size="${p['sensors']['mid360']['visual_proxy']['mount_size_m'][0]} ${p['sensors']['mid360']['visual_proxy']['mount_size_m'][1]} ${p['sensors']['mid360']['visual_proxy']['mount_size_m'][2]}"/>
+      </geometry>
+      <material name="mid360_mount_gray"/>
+    </visual>
+    <visual name="mid360_body_visual">
+      <origin xyz="0 0 ${p['sensors']['mid360']['visual_proxy']['mount_size_m'][2] + p['sensors']['mid360']['visual_proxy']['body_size_m'][2] / 2.0}" rpy="0 0 0"/>
+      <geometry>
+        <box size="${p['sensors']['mid360']['visual_proxy']['body_size_m'][0]} ${p['sensors']['mid360']['visual_proxy']['body_size_m'][1]} ${p['sensors']['mid360']['visual_proxy']['body_size_m'][2]}"/>
+      </geometry>
+      <material name="mid360_body_gray"/>
+    </visual>
+    <visual name="mid360_scan_window_visual">
+      <origin xyz="0 0 ${lidar_housing_height - p['sensors']['mid360']['visual_proxy']['scan_window_height_m'] / 2.0}" rpy="0 0 0"/>
       <geometry>
         <cylinder
-          radius="${p['sensors']['mid360']['visual_proxy']['radius_m']}"
-          length="${lidar_housing_height}"/>
-      </geometry>
-      <material name="sensor_gray"/>
+          radius="${p['sensors']['mid360']['visual_proxy']['scan_window_radius_m']}"
+          length="${p['sensors']['mid360']['visual_proxy']['scan_window_height_m']}"/>
+      </geometry>
+      <material name="mid360_window_black"/>
     </visual>
   </link>
