Commit message: fix(description): keep MID-360 visual proxy out of the hashed sensor section
57e602b replaced sensors.mid360.visual_proxy.radius_m with visual-only
envelope sizes. sensors.mid360 is hashed into extrinsics_hash, so the
accepted Issue #13 and Issue #53 motion profiles were rejected and
start_auto_nav.sh stopped with MOTION_PROFILE_REJECTED, although no real
extrinsic changed.

Move the envelope sizes to geometry.mid360_visual_proxy and restore the
legacy radius_m in sensors.mid360, so extrinsics_hash is again
7691c3c2... and both accepted profiles pass check_motion_profile.py and
check_linear_profile.py.

Co-Authored-By: Claude Opus 5.5 <noreply@anthropic.com>

File: src/carbot_description/urdf/carbot.urdf.xacro (robot description, xacro)
@@ -155,23 +155,23 @@
          remain defined by the fixed joints and canonical calibration above. -->
     <visual name="mid360_mount_visual">
-      <origin xyz="0 0 ${p['sensors']['mid360']['visual_proxy']['mount_size_m'][2] / 2.0}" rpy="0 0 0"/>
-      <geometry>
-        <box size="${p['sensors']['mid360']['visual_proxy']['mount_size_m'][0]} ${p['sensors']['mid360']['visual_proxy']['mount_size_m'][1]} ${p['sensors']['mid360']['visual_proxy']['mount_size_m'][2]}"/>
+      <origin xyz="0 0 ${p['geometry']['mid360_visual_proxy']['mount_size_m'][2] / 2.0}" rpy="0 0 0"/>
+      <geometry>
+        <box size="${p['geometry']['mid360_visual_proxy']['mount_size_m'][0]} ${p['geometry']['mid360_visual_proxy']['mount_size_m'][1]} ${p['geometry']['mid360_visual_proxy']['mount_size_m'][2]}"/>
       </geometry>
       <material name="mid360_mount_gray"/>
     </visual>
     <visual name="mid360_body_visual">
-      <origin xyz="0 0 ${p['sensors']['mid360']['visual_proxy']['mount_size_m'][2] + p['sensors']['mid360']['visual_proxy']['body_size_m'][2] / 2.0}" rpy="0 0 0"/>
-      <geometry>
-        <box size="${p['sensors']['mid360']['visual_proxy']['body_size_m'][0]} ${p['sensors']['mid360']['visual_proxy']['body_size_m'][1]} ${p['sensors']['mid360']['visual_proxy']['body_size_m'][2]}"/>
+      <origin xyz="0 0 ${p['geometry']['mid360_visual_proxy']['mount_size_m'][2] + p['geometry']['mid360_visual_proxy']['body_size_m'][2] / 2.0}" rpy="0 0 0"/>
+      <geometry>
+        <box size="${p['geometry']['mid360_visual_proxy']['body_size_m'][0]} ${p['geometry']['mid360_visual_proxy']['body_size_m'][1]} ${p['geometry']['mid360_visual_proxy']['body_size_m'][2]}"/>
       </geometry>
       <material name="mid360_body_gray"/>
     </visual>
     <visual name="mid360_scan_window_visual">
-      <origin xyz="0 0 ${lidar_housing_height - p['sensors']['mid360']['visual_proxy']['scan_window_height_m'] / 2.0}" rpy="0 0 0"/>
+      <origin xyz="0 0 ${lidar_housing_height - p['geometry']['mid360_visual_proxy']['scan_window_height_m'] / 2.0}" rpy="0 0 0"/>
       <geometry>
         <cylinder
-          radius="${p['sensors']['mid360']['visual_proxy']['scan_window_radius_m']}"
-          length="${p['sensors']['mid360']['visual_proxy']['scan_window_height_m']}"/>
+          radius="${p['geometry']['mid360_visual_proxy']['scan_window_radius_m']}"
+          length="${p['geometry']['mid360_visual_proxy']['scan_window_height_m']}"/>
       </geometry>
       <material name="mid360_window_black"/>
